File: v0.2/Kimiro.kicad_pcb (KiCad board)
At the start: 2 copper layers, 17.8 x 33.1 mm, 27 parts, among them J1 Conn_01x04, J2 USB_C_Left, J3 Left, J4 Right, Q1 AO3407, U1 TP4054, U3 MS88FS3, U4 XC6220B331MR

Commit message: Cập nhật file PCB
Parts:
- added REF**7: breakaway-mousebites, Kimiro-library:breakaway-mousebites, F.Cu at (86.4, 60.9)
- added REF**7: breakaway-mousebites, Kimiro-library:breakaway-mousebites, F.Cu at (76.2, 67.4)
- added REF**7: breakaway-mousebites, Kimiro-library:breakaway-mousebites, F.Cu at (86.4, 38.2)
- added kibuzzard-62E2A6C4: G***, kibuzzard-62E2A6C4, B.Cu at (76.2, 61.6)
- moved kibuzzard-62E129EE 0.05 mm to (77.5, 65.0)
Connections:
- U3 pad 10: unconnected-(U3-Pad10) -> 100
- U3 pad 11: unconnected-(U3-Pad11) -> 024
- U3 pad 12: unconnected-(U3-Pad12) -> 020
- U3 pad 13: unconnected-(U3-Pad13) -> 021
Routing:
- net 020: track 2.97 -> 15.8 mm
- net 021: track 3.09 -> 15.5 mm
- net 024: track 7.22 -> 19.3 mm
- net 100: track 9.09 -> 21.0 mm
- net GND: track 28.0 -> 35.0 mm, vias 5 -> 6
- net SWCLK: track 4.50 -> 3.88 mm
- removed copper zone on B.Cu, net (none)
- removed copper zone on F.Cu, net (none)
Other:
- board size 17.8 x 33.1 mm -> 20.3 x 35.6 mm
- board text removed: "KIMIRO"
