File: PCB/nRFpill/v0.2/nRFpill.kicad_sch (KiCad schematic)
At the start: 33 parts, among them J1 USB_C_Receptacle_USB2.0, J2 , J3 , J4 , J5 , Q1 AO3407, Q2 AO3407, SW1 RST, SW2 DFU, U1 MIC5219-3.3YM5, U2 USBLC6-2SC6, U3 TP4054, U5 MS88FS3

Commit message: Update nRFpill
Parts:
- removed D4: BLUE, LED_SMD:LED_0603_1608Metric, symbol Device:LED
- removed R11: 1K, Resistor_SMD:R_0603_1608Metric, symbol Device:R_Small
- C5: value 0.1uF -> 100nF
- J1: footprint kien242:USB-C-16pin-hight -> kien242:USB-C-Low
- R10: value RPROG -> 2.3k
- R6: value 2M -> 100k
- U5: footprint kien242:MS88SF3-nRF52840 -> kien242:MODULE_MS88SF3
Connections:
- net LED_2 is gone; now on net 0.24: U5.60 (1.03)
- net 0.05: now also J3.15 (Pin_15); no longer J3.14 (Pin_14)
- net 0.27: now also J3.14 (Pin_14); no longer J3.15 (Pin_15)
- net 1.00: now also U5.59 (1.01)
- net DFU: now also U5.56 (0.10); no longer U5.59 (1.01)
- net LED_1: now also U5.2 (1.11); no longer U5.58 (1.05)
- net POWER_PIN: now also U5.58 (1.05)
- net SWDIO: now also U5.57 (1.07)
- net 009: now reaches U5.55 (0.09)
- net 009: now also J2.1 (Pin_1)
- removed net 1.07: J2.1 (Pin_1), U5.57 (1.07)
