File: PCB/Kimiro/v0.3/Kimiro.kicad_pcb (KiCad board)
At the start: 2 copper layers, 17.8 x 33.1 mm, 44 parts, among them J1 USB_C_Left, J2 Left, J3 Right, J4 , J5 , J6 , Q1 AO3407, U1 TP4054, U2 MS88FS3, U3 XC6220B331MR

Commit message: Update bootloader.hex, flashbed.kicad_pcb, and 54 more files...
Parts:
- removed kibuzzard-62E129EE: G***, kibuzzard-62E129EE
- removed kibuzzard-635CFD08: G***, kibuzzard-635CFD08
- removed kibuzzard-635CFD0E: G***, kibuzzard-635CFD0E
- added J7: , Kimiro-library:Conn_1x01, B.Cu at (72.4, 52.1)
- added J8: , Kimiro-library:Conn_1x01, B.Cu at (80.0, 52.1)
- added kibuzzard-63BCF8A2: G***, kibuzzard-63BCF8A2, B.Cu at (74.9, 49.8)
- added kibuzzard-63BCF8A9: G***, kibuzzard-63BCF8A9, B.Cu at (77.5, 49.8)
- added kibuzzard-63BCF8C7: G***, kibuzzard-63BCF8C7, B.Cu at (72.4, 49.4)
- added kibuzzard-640324C5: G***, kibuzzard-640324C5, B.Cu at (80.0, 49.8)
- added kibuzzard-64034CD4: G***, kibuzzard-64034CD4, B.Cu at (76.7, 64.8)
- moved kibuzzard-635D09C5 0.41 mm to (73.2, 63.0)
- moved kibuzzard-62E2A6C4 0.15 mm to (76.2, 61.5)
Connections:
- J5 pad 1: SWCLK -> SWDIO
- J6 pad 1: SWDIO -> SWCLK
Routing:
- net VDD: track 6.99 -> 10.3 mm
- net SWCLK: track 9.05 -> 12.0 mm
- net 008: track 16.6 -> 18.1 mm
- net 109: track 19.4 -> 20.9 mm
- net 007: track 14.6 -> 15.8 mm
- net SWDIO: track 11.4 -> 10.3 mm
- net 027: track 6.74 -> 7.64 mm
- net 013: track 16.9 -> 17.6 mm
- net 017: track 8.23 -> 7.67 mm
- net D-: track 15.6 -> 16.2 mm
Other:
- board text added: "007"
- board text removed: "108"
